File: card.kicad_pcb (KiCad board)
At the start: 2 copper layers, 85.6 x 54 mm, 10 parts

Commit message: cleaning up layout
Parts:
- removed the G*** at (56.2, 68.7) (x5)
- added Ref**: Val**, custom-footprints:globered, F.Cu at (56.3, 68.7)
